Commit message: messy

File: src/my_robot_description/xacro/camera.xacro (robot description, xacro)
@@ -2,9 +2,30 @@
 <robot xmlns:xacro="http://www.ros.org/wiki/xacro">
     <joint name="camera_joint" type="fixed">
-        <parent link="chassis"/>
+        <parent link="base_link"/>
         <child link="camera_link"/>
-        <origin xyz="0.4 0 0.65" rpy="0 0 0"/>
+        <origin xyz="0.25 0 1.01" rpy="0 0.6283 0"/>
+    </joint>
+    <joint name="camera_joint_rear" type="fixed">
+        <parent link="base_link"/>
+        <child link="camera_link_rear"/>
+        <origin xyz="0.381 0 1.14" rpy="0 0.5934 ${pi}"/>
     </joint>
     <link name="camera_link">
+        <visual>
+            <geometry>
+                <box size="0.010 0.03 0.03"/>
+            </geometry>
+            <material name="red"/>
+        </visual>
+        <collision>
+            <geometry>
+                <box size="0.010 0.03 0.03"/>
+            </geometry>
+        </collision>
+        <xacro:inertial_box mass="0.1" x="0.01" y="0.3" z="0.3">
+            <origin xyz="0 0 0" rpy="0 0 0"/>
+        </xacro:inertial_box>
+    </link>
+    <link name="camera_link_rear">
         <visual>
             <geometry>
@@ -28,4 +49,10 @@
     </joint>
     <link name="camera_link_optical"></link>
+    <joint name="camera_optical_joint_rear" type="fixed">
+        <parent link="camera_link_rear"/>
+        <child link="camera_link_optical_rear"/>
+        <origin xyz="0 0 0" rpy="${-pi/2} 0 ${-pi/2}"/>
+    </joint>
+    <link name="camera_link_optical_rear"></link>
     <xacro:if value="$(arg sim_mode)">
         <gazebo reference="camera_link">

File: src/my_robot_description/xacro/lidar_3d.xacro (robot description, xacro)
@@ -2,7 +2,7 @@
 <robot xmlns:xacro="http://www.ros.org/wiki/xacro">
     <joint name="lidar_joint" type="fixed">
-        <parent link="chassis"/>
+        <parent link="base_link"/>
         <child link="lidar_frame"/>
-        <origin xyz="0.305 0 0.71" rpy="0 0 0"/>
+        <origin xyz="0.29 0 0.3048" rpy="0 0 ${pi}"/>
     </joint>
     <link name="lidar_frame">
@@ -22,4 +22,10 @@
         </xacro:inertial_cylinder>
     </link>
+    <joint name="lidar_frame_to_os_sensor" type="fixed">
+        <parent link="lidar_frame"/>
+        <child link="os_sensor"/>
+        <origin xyz="0 0 0" rpy="0 0 0"/>
+    </joint>
+    <link name="os_sensor"/>
     <xacro:if value="$(arg sim_mode)">
         <gazebo reference="lidar_frame">

Commit message: Update information not tracked.

File: src/my_robot_description/xacro/camera.xacro (robot description, xacro)
@@ -4,10 +4,10 @@
         <parent link="base_link"/>
         <child link="camera_link"/>
-        <origin xyz="0.25 0 1.01" rpy="0 0.6283 0"/>
+        <origin xyz="0.25 0 1.14" rpy="0 0.6283 0"/>
     </joint>
     <joint name="camera_joint_rear" type="fixed">
         <parent link="base_link"/>
         <child link="camera_link_rear"/>
-        <origin xyz="0.381 0 1.14" rpy="0 0.5934 ${pi}"/>
+        <origin xyz="0.381 0 1.01" rpy="0 0.5934 ${pi}"/>
     </joint>
     <link name="camera_link">

Commit message: Fix xacro, test camera and lane detection.

File: src/my_robot_description/xacro/camera.xacro (robot description, xacro)
@@ -3,13 +3,15 @@
     <joint name="camera_joint" type="fixed">
         <parent link="base_link"/>
-        <child link="camera_link"/>
-        <origin xyz="0.25 0 1.14" rpy="0 0.6283 0"/>
+        <child link="zed_camera_link"/>
+        <origin xyz="0.381 0 1.01" rpy="0 0.6283 0"/>
     </joint>
     <joint name="camera_joint_rear" type="fixed">
         <parent link="base_link"/>
-        <child link="camera_link_rear"/>
-        <origin xyz="0.381 0 1.01" rpy="0 0.5934 ${pi}"/>
+        <child link="zed_rear_camera_link"/>
+        <origin xyz="0.25 0 1.14" rpy="0 0.5934 ${pi}"/>
     </joint>
-    <link name="camera_link">
+    <link name="zed_camera_link"></link>
+    <link name="zed_rear_camera_link"></link>
+    <!-- <link name="camera_link">
         <visual>
             <geometry>
@@ -42,6 +44,6 @@
             <origin xyz="0 0 0" rpy="0 0 0"/>
         </xacro:inertial_box>
-    </link>
-    <joint name="camera_optical_joint" type="fixed">
+    </link> -->
+    <!-- <joint name="camera_optical_joint" type="fixed">
         <parent link="camera_link"/>
         <child link="camera_link_optical"/>
@@ -54,5 +56,5 @@
         <origin xyz="0 0 0" rpy="${-pi/2} 0 ${-pi/2}"/>
     </joint>
-    <link name="camera_link_optical_rear"></link>
+    <link name="camera_link_optical_rear"></link> -->
     <xacro:if value="$(arg sim_mode)">
         <gazebo reference="camera_link">
