Commit message: Update.

File: src/my_robot_description/xacro/gps.xacro (robot description, xacro)
@@ -4,5 +4,5 @@
         <parent link="base_link"/>
         <child link="gps_link"/>
-        <origin xyz="0 0 0.1" rpy="0 0 0"/>
+        <origin xyz="0.34 0 1.21" rpy="0 0 0"/>
     </joint>
     <link name="gps_link">
